File: schematic/fiendPrototype.kicad_sch (KiCad schematic)
At the start: 9 parts

Commit message: docs: add comment to schematic
Other:
- company: (none) -> Oscar Peace
- title: (none) -> Fiend Prototype
Changed lines of the file:
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@@
 	(generator_version "8.0")
 	(paper "A4")
+	(title_block
+		(title "Fiend Prototype")
+		(date "2024-08-30")
+		(company "Oscar Peace")
+		(comment 1 "Don't make one of these yourself.")
+	)
 	(junction
 		(at 194.31 116.84)
